File: Schematic/onboard_v1.0.sch (EAGLE design)
At the start: 26 parts

Commit message: Latest schematic update
Parts:
- removed R3, R4, R5, R6: (no value), rcl:POTENTIOMETER_PT-10
- added R10, R7, R8, R9: (no value), rcl:POTENTIOMETER_PT-10
- added U$16: IL-MATTO, ganges:IL-MATTO
Connections:
- new net GND_A1: U$16.GND_A
- new net GND_A_1: R10.2, R7.2, R8.2, R9.2
- new net ILM_TO_LEO: PCB1.0(RX), U$1.PD1
- new net LEO_TO_ILM: PCB1.1(TX), U$1.PD0
- new net POT1_X: R7.3, U$16.PA0
- new net POT1_Y: R10.3, U$16.PA1
- new net POT2_X: R8.3, U$16.PA2
- new net POT2_Y: R9.3, U$16.PA3
- new net V_A_1: R10.1, R7.1, R8.1, R9.1, U$16.V_A
Other:
- moved on the sheet: R1, R2, S1, S2, S3, S4
Changed lines of the file:
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@@
 <part name="R1" library="rcl" deviceset="R-EU_" device="0204/7"/>
 <part name="R2" library="rcl" deviceset="R-EU_" device="0204/7"/>
-<part name="R3" library="rcl" deviceset="POTENTIOMETER_" device="PT-10"/>
-<part name="R4" library="rcl" deviceset="POTENTIOMETER_" device="PT-10"/>
-<part name="R5" library="rcl" deviceset="POTENTIOMETER_" device="PT-10"/>
-<part name="R6" library="rcl" deviceset="POTENTIOMETER_" device="PT-10"/>
 <part name="S1" library="switch" deviceset="320-916" device=""/>
 <part name="S2" library="switch" deviceset="320-916" device=""/>
@@
 <part name="U$14" library="ganges" deviceset="RFM12B-S2" device=""/>
 <part name="U$15" library="ganges" deviceset="GND" device=""/>
+<part name="U$16" library="ganges" deviceset="IL-MATTO" device=""/>
+<part name="R7" library="rcl" deviceset="POTENTIOMETER_" device="PT-10"/>
+<part name="R8" library="rcl" deviceset="POTENTIOMETER_" device="PT-10"/>
+<part name="R9" library="rcl" deviceset="POTENTIOMETER_" device="PT-10"/>
+<part name="R10" library="rcl" deviceset="POTENTIOMETER_" device="PT-10"/>
 </parts>
 <sheets>
@@
 </plain>
 <instances>
-<instance part="PCB1" gate="G$1" x="83.82" y="60.96"/>
-<instance part="U$1" gate="G$1" x="-104.14" y="78.74"/>
+<instance part="PCB1" gate="G$1" x="88.9" y="-7.62"/>
+<instance part="U$1" gate="G$1" x="-66.04" y="5.08"/>
 <instance part="U$2" gate="G$1" x="160.02" y="55.88"/>
-<instance part="U$3" gate="G$1" x="7.62" y="35.56"/>
-<instance part="U$4" gate="G$1" x="7.62" y="2.54"/>
-<instance part="U$5" gate="G$1" x="7.62" y="101.6"/>
-<instance part="R1" gate="G$1" x="-127" y="68.58"/>
-<instance part="R2" gate="G$1" x="-127" y="76.2"/>
-<instance part="R3" gate="1" x="-127" y="33.02"/>
-<instance part="R4" gate="1" x="-127" y="45.72"/>
-<instance part="R5" gate="1" x="-127" y="58.42"/>
-<instance part="R6" gate="1" x="-127" y="88.9"/>
-<instance part="S1" gate="1" x="-99.06" y="40.64"/>
-<instance part="S2" gate="1" x="-99.06" y="22.86"/>
-<instance part="S3" gate="1" x="-99.06" y="5.08"/>
-<instance part="S4" gate="1" x="-99.06" y="55.88"/>
-<instance part="U$6" gate="G$1" x="7.62" y="60.96"/>
+<instance part="U$3" gate="G$1" x="101.6" y="53.34"/>
+<instance part="U$4" gate="G$1" x="93.98" y="137.16"/>
+<instance part="U$5" gate="G$1" x="58.42" y="-71.12"/>
+<instance part="R1" gate="G$1" x="152.4" y="144.78"/>
+<instance part="R2" gate="G$1" x="152.4" y="152.4"/>
+<instance part="S1" gate="1" x="40.64" y="213.36"/>
+<instance part="S2" gate="1" x="43.18" y="193.04"/>
+<instance part="S3" gate="1" x="40.64" y="177.8"/>
+<instance part="S4" gate="1" x="38.1" y="226.06"/>
+<instance part="U$6" gate="G$1" x="-53.34" y="-60.96"/>
 <instance part="U$7" gate="G$1" x="236.22" y="68.58"/>
 <instance part="U$8" gate="G$1" x="160.02" y="25.4"/>
@@
 <instance part="U$12" gate="G$1" x="236.22" y="7.62"/>
 <instance part="U$13" gate="G$1" x="236.22" y="-22.86"/>
-<instance part="U$14" gate="G$1" x="7.62" y="78.74"/>
+<instance part="U$14" gate="G$1" x="17.78" y="137.16"/>
 <instance part="U$15" gate="G$1" x="142.24" y="-43.18"/>
+<instance part="U$16" gate="G$1" x="-91.44" y="88.9"/>
+<instance part="R7" gate="1" x="17.78" y="208.28"/>
+<instance part="R8" gate="1" x="0" y="205.74"/>
+<instance part="R9" gate="1" x="0" y="215.9"/>
+<instance part="R10" gate="1" x="17.78" y="218.44"/>
 </instances>
 <busses>
@@
 </segment>
 </net>
+<net name="POT1_X" class="0">
+<segment>
+<pinref part="R7" gate="1" pin="3"/>
+<wire x1="17.78" y1="203.2" x2="17.78" y2="193.04" width="0.1524" layer="91"/>
+<wire x1="17.78" y1="193.04" x2="-15.24" y2="193.04" width="0.1524" layer="91"/>
+<label x="-15.24" y="193.04" size="1.27" layer="95" rot="R180" xref="yes"/>
+</segment>
+<segment>
+<pinref part="U$16" gate="G$1" pin="PA0"/>
+<wire x1="-7.62" y1="157.48" x2="-7.62" y2="162.56" width="0.1524" layer="91"/>
+<label x="-7.62" y="162.56" size="1.27" layer="95" rot="R90" xref="yes"/>
+</segment>
+</net>
+<net name="POT1_Y" class="0">
+<segment>
+<wire x1="10.16" y1="195.58" x2="-15.24" y2="195.58" width="0.1524" layer="91"/>
+<pinref part="R10" gate="1" pin="3"/>
+<wire x1="17.78" y1="213.36" x2="10.16" y2="213.36" width="0.1524" layer="91"/>
+<wire x1="10.16" y1="213.36" x2="10.16" y2="195.58" width="0.1524" layer="91"/>
+<label x="-15.24" y="195.58" size="1.27" layer="95" rot="R180" xref="yes"/>
+</segment>
+<segment>
+<pinref part="U$16" gate="G$1" pin="PA1"/>
+<wire x1="-10.16" y1="157.48" x2="-10.16" y2="162.56" width="0.1524" layer="91"/>
+<label x="-10.16" y="162.56" size="1.27" layer="95" rot="R90" xref="yes"/>
+</segment>
+</net>
+<net name="POT2_X" class="0">
+<segment>
+<pinref part="R8" gate="1" pin="3"/>
+<wire x1="0" y1="200.66" x2="0" y2="198.12" width="0.1524" layer="91"/>
+<wire x1="0" y1="198.12" x2="-15.24" y2="198.12" width="0.1524" layer="91"/>
+<label x="-15.24" y="198.12" size="1.27" layer="95" rot="R180" xref="yes"/>
+</segment>
+<segment>
+<pinref part="U$16" gate="G$1" pin="PA2"/>
+<wire x1="-12.7" y1="157.48" x2="-12.7" y2="162.56" width="0.1524" layer="91"/>
+<label x="-12.7" y="162.56" size="1.27" layer="95" rot="R90" xref="yes"/>
+</segment>
+</net>
+<net name="POT2_Y" class="0">
+<segment>
+<pinref part="R9" gate="1" pin="3"/>
+<wire x1="0" y1="210.82" x2="-7.62" y2="210.82" width="0.1524" layer="91"/>
+<wire x1="-7.62" y1="210.82" x2="-7.62" y2="200.66" width="0.1524" layer="91"/>
+<wire x1="-7.62" y1="200.66" x2="-15.24" y2="200.66" width="0.1524" layer="91"/>
+<label x="-15.24" y="200.66" size="1.27" layer="95" rot="R180" xref="yes"/>
+</segment>
+<segment>
+<pinref part="U$16" gate="G$1" pin="PA3"/>
+<wire x1="-15.24" y1="157.48" x2="-15.24" y2="162.56" width="0.1524" layer="91"/>
+<label x="-15.24" y="162.56" size="1.27" layer="95" rot="R90" xref="yes"/>
+</segment>
+</net>
+<net name="GND_A_1" class="0">
+<segment>
+<wire x1="-15.24" y1="220.98" x2="5.08" y2="220.98" width="0.1524" layer="91"/>
+<pinref part="R9" gate="1" pin="2"/>
+<wire x1="5.08" y1="220.98" x2="5.08" y2="215.9" width="0.1524" layer="91"/>
+<wire x1="5.08" y1="220.98" x2="22.86" y2="220.98" width="0.1524" layer="91"/>
+<junction x="5.08" y="220.98"/>
+<pinref part="R10" gate="1" pin="2"/>
+<wire x1="22.86" y1="220.98" x2="22.86" y2="218.44" width="0.1524" layer="91"/>
+<pinref part="R7" gate="1" pin="2"/>
+<wire x1="22.86" y1="218.44" x2="22.86" y2="208.28" width="0.1524" layer="91"/>
+<junction x="22.86" y="218.44"/>
+<pinref part="R8" gate="1" pin="2"/>
+<wire x1="5.08" y1="215.9" x2="5.08" y2="205.74" width="0.1524" layer="91"/>
+<junction x="5.08" y="215.9"/>
+<label x="-15.24" y="220.98" size="1.27" layer="95" rot="R180" xref="yes"/>
+</segment>
+</net>
+<net name="GND_A1" class="0">
+<segment>
+<pinref part="U$16" gate="G$1" pin="GND_A"/>
+<wire x1="-35.56" y1="157.48" x2="-35.56" y2="162.56" width="0.1524" layer="91"/>
+<label x="-35.56" y="162.56" size="1.27" layer="95" rot="R90" xref="yes"/>
+</segment>
+</net>
+<net name="V_A_1" class="0">
+<segment>
+<pinref part="U$16" gate="G$1" pin="V_A"/>
+<wire x1="-33.02" y1="157.48" x2="-33.02" y2="162.56" width="0.1524" layer="91"/>
+<label x="-33.02" y="162.56" size="1.27" layer="95" rot="R90" xref="yes"/>
+</segment>
+<segment>
+<pinref part="R9" gate="1" pin="1"/>
+<pinref part="R8" gate="1" pin="1"/>
+<wire x1="-10.16" y1="215.9" x2="-5.08" y2="215.9" width="0.1524" layer="91"/>
+<wire x1="-10.16" y1="215.9" x2="-10.16" y2="205.74" width="0.1524" layer="91"/>
+<wire x1="-10.16" y1="205.74" x2="-5.08" y2="205.74" width="0.1524" layer="91"/>
+<wire x1="-10.16" y1="215.9" x2="-10.16" y2="218.44" width="0.1524" layer="91"/>
+<wire x1="-10.16" y1="218.44" x2="-15.24" y2="218.44" width="0.1524" layer="91"/>
+<junction x="-10.16" y="215.9"/>
+<pinref part="R10" gate="1" pin="1"/>
+<wire x1="-10.16" y1="218.44" x2="7.62" y2="218.44" width="0.1524" layer="91"/>
+<junction x="-10.16" y="218.44"/>
+<pinref part="R7" gate="1" pin="1"/>
+<wire x1="7.62" y1="218.44" x2="12.7" y2="218.44" width="0.1524" layer="91"/>
+<wire x1="12.7" y1="208.28" x2="7.62" y2="208.28" width="0.1524" layer="91"/>
+<wire x1="7.62" y1="208.28" x2="7.62" y2="218.44" width="0.1524" layer="91"/>
+<junction x="7.62" y="218.44"/>
+<label x="-15.24" y="218.44" size="1.27" layer="95" rot="R180" xref="yes"/>
+</segment>
+</net>
+<net name="LEO_TO_ILM" class="0">
+<segment>
+<pinref part="U$1" gate="G$1" pin="PD0"/>
+<wire x1="-50.8" y1="0" x2="-50.8" y2="-5.08" width="0.1524" layer="91"/>
+<label x="-50.8" y="-5.08" size="1.27" layer="95" rot="R270" xref="yes"/>
+</segment>
+<segment>
+<pinref part="PCB1" gate="G$1" pin="1(TX)"/>
+<wire x1="111.76" y1="15.24" x2="111.76" y2="20.32" width="0.1524" layer="91"/>
+<label x="111.76" y="20.32" size="1.27" layer="95" rot="R90" xref="yes"/>
+</segment>
+</net>
+<net name="ILM_TO_LEO" class="0">
+<segment>
+<pinref part="U$1" gate="G$1" pin="PD1"/>
+<wire x1="-48.26" y1="0" x2="-48.26" y2="-5.08" width="0.1524" layer="91"/>
+<label x="-48.26" y="-5.08" size="1.27" layer="95" rot="R270" xref="yes"/>
+</segment>
+<segment>
+<pinref part="PCB1" gate="G$1" pin="0(RX)"/>
+<wire x1="114.3" y1="15.24" x2="114.3" y2="20.32" width="0.1524" layer="91"/>
+<label x="114.3" y="20.32" size="1.27" layer="95" rot="R90" xref="yes"/>
+</segment>
+</net>

Commit message: Update of System schematic
Parts:
- added LEFT_FRONT_ESC: ESC, ganges:ESC
- U$2: value ESC -> VCC; device ganges:ESC -> ganges:VCC
- renumbered U$10 to RIGHT_REAR_ESC, U$11 to RIGHT_FRONT_MOTOR, U$12 to LEFT_REAR_MOTOR, U$13 to RIGHT_REAR_MOTOR, U$7 to LEFT_FRONT_MOTOR, U$8 to RIGHT_FRONT_ESC, U$9 to LEFT_REAR_ESC
Connections:
- removed net GND_A1: U$16.GND_A
- removed net N$13: LEFT_REAR_ESC.GND_CONTROL, LEFT_REAR_ESC.GND_IN, RIGHT_FRONT_ESC.GND_CONTROL, RIGHT_FRONT_ESC.GND_IN, RIGHT_REAR_ESC.GND_CONTROL, RIGHT_REAR_ESC.GND_IN, U$2.GND_CONTROL, U$2.GND_IN
- new net 11.1V_LIPO: LEFT_FRONT_ESC.V_IN, LEFT_REAR_ESC.V_IN, RIGHT_FRONT_ESC.V_IN, RIGHT_REAR_ESC.V_IN, U$2.VCC
- new net ANT_BASE: U$14.ANT
- new net ANT_UAV: U$5.ANT
- new net GND_A_2: U$1.GND_A, U$4.GND
- new net GND_B_1: U$14.GND, U$16.GND_B
- new net GND_B_2: U$1.GND_B, U$5.GND
- new net GND_D_2: U$1.GND_D, U$6.GND
- new net GND_EXT_2: PCB1.GND.., U$1.GND_EXT
- new net GND_LEO: U$3.GND
- new net GND_LIPO: LEFT_FRONT_ESC.GND_CONTROL, LEFT_FRONT_ESC.GND_IN, LEFT_REAR_ESC.GND_CONTROL, LEFT_REAR_ESC.GND_IN, RIGHT_FRONT_ESC.GND_CONTROL, RIGHT_FRONT_ESC.GND_IN, RIGHT_REAR_ESC.GND_CONTROL, RIGHT_REAR_ESC.GND_IN
- new net ILM_TO_PC(YEL): U$16.PD1
- new net INT: PCB1.7, U$3.INT
- new net IR_DATA: U$1.PA0, U$4.DATA
- new net LEFT_FRONT: LEFT_FRONT_ESC.CONTROL_IN, PCB1.~9
- new net LEFT_REAR: LEFT_REAR_ESC.CONTROL_IN, PCB1.~11
- new net NIRQ_BASE: U$14.IRQ, U$16.PD3
- new net NIRQ_UAV: U$1.PD3, U$5.IRQ
- new net NSEL_BASE: U$14.SEL, U$16.PB4
- new net NSEL_UAV: U$1.PB4, U$5.SEL
- new net PC_TO_ILM(ORNG): U$16.PD0
- new net RIGHT_FRONT: PCB1.~10, RIGHT_FRONT_ESC.CONTROL_IN
- new net RIGHT_REAR: PCB1.~5, RIGHT_REAR_ESC.CONTROL_IN
- new net SCK_BASE: U$14.SCK, U$16.PB7
- new net SCK_UAV: U$1.PB7, U$5.SCK
- new net SCL: PCB1.18(SCL), U$3.SCL
- new net SDA: PCB1.19(SDA), U$3.SDA
- new net SDI_BASE: U$14.SDI, U$16.PB5
- new net SDI_UAV: U$1.PB5, U$5.SDI
- new net SDO_BASE: U$14.SDO, U$16.PB6
- new net SDO_UAV: U$1.PB6, U$5.SDO
- new net SERVO_CONTROL: U$1.PD7, U$6.CONTROL
- new net V_A_2: U$1.V_A, U$4.VCC
- new net V_B_1: U$14.VCC, U$16.V_B
- new net V_B_2: U$1.V_B, U$5.VCC
- new net V_D_2: U$1.V_D, U$6.VCC
- new net V_EXT_2: PCB1.5V, U$1.V_EXT
- new net V_LEO: U$3.VCC
- net GND_A_1: now also U$16.GND_A
- net N$1: now also LEFT_FRONT_ESC.OUT_A; no longer U$2.OUT_A
- net N$2: now also LEFT_FRONT_ESC.OUT_B; no longer U$2.OUT_B
- net N$3: now also LEFT_FRONT_ESC.OUT_C; no longer U$2.OUT_C

Commit message: Finalised first version of low level schematic
Parts:
- removed U$15: GND, ganges:GND
- removed U$2: VCC, ganges:VCC
Connections:
- net INT renamed GYRO_INT
- net IR_DATA renamed ADC_IR
- net POT1_X renamed ADC_POT1_X
- net POT1_Y renamed ADC_POT1_Y
- net POT2_X renamed ADC_POT2_X
- net POT2_Y renamed ADC_POT2_Y
- net SCL renamed GYRO_SCL
- net SDA renamed GYRO_SDA
- new net ADC_BATT: R1.1, R2.2, U$1.PA1
- new net GND_C_1: S1.O, S2.O, S3.O, S4.O, U$16.GND_C
- new net SW0: S1.P, U$16.PC0
- new net SW1: S2.P, U$16.PC1
- new net SW2: S3.P, U$16.PC2
- new net SW3: S4.P, U$16.PC3
- new net V_C_1: S1.S, S2.S, S3.S, S4.S, U$16.V_C
- net 11.1V_LIPO: now also PCB1.VIN, R1.2; no longer U$2.VCC
- net GND_LIPO: now also PCB1.GND., R2.1
Other:
- note added: "06/03/17"
- note added: "Arduino"
- note added: "Base"
- note added: "Base Il Matto"
- note added: "Base Transceiver"
- note added: "Batt Lvl"
- note added: "Ben Rowlinson Lawrence Gray Joel Trickey Joseph Hindmarsh Mohammed Ibrahim"
- note added: "Control Pots"
- note added: "Control Switches"
- note added: "IMU"
- note added: "IR"
- note added: "Motor Control"
- note added: "Servo"
- note added: "Team Ganges Low Level Schematic"
- note added: "UAV"
- note added: "UAV Il Matto"
- note added: "UAV Transceiver"
- moved on the sheet: R1, R10, R2, R7, R8, R9, S1, S2, S3, S4
