File: Schematic/onboard_v1.1.sch (EAGLE design)
At the start: 29 parts

Commit message: Absolute FINAL SCHEMATIC
Parts:
- C1: value (none) -> 0.1u
- C2: value (none) -> 100u
Other:
- note added: "15/03/17"
- note added: "PDB"
- note added: "Team Ganges Low Level Schematic v1.1"
- note removed: "06/03/17"
- note removed: "Team Ganges Low Level Schematic"
- moved on the sheet: C1, C2
